Commit message: Fix: Make everything a lot more functional

File: src/robot_description/urdf/robot.urdf (robot description, URDF)
Before this commit: robot simple_robot, 6 links, 5 joints
Joints:
- joint joint_wheel_front_left: axis 0 1 0 -> 0 0 1
- joint joint_wheel_front_right: axis 0 1 0 -> 0 0 1
- joint joint_wheel_rear_left: axis 0 1 0 -> 0 0 1
- joint joint_wheel_rear_right: axis 0 1 0 -> 0 0 1

File: src/robot_description/urdf/robot.urdf.xacro (robot description, xacro)
@@ -1,32 +1,44 @@
 <?xml version="1.0"?>
-<robot name="simple_robot" xmlns:xacro="http://www.ros.org/wiki/xacro">
-  <!-- Materials -->
+<robot name="mobile_robot" xmlns:xacro="http://www.ros.org/wiki/xacro">
+  <xacro:property name="chassis_length" value="0.6" />
+  <xacro:property name="chassis_width" value="0.5" />
+  <xacro:property name="chassis_height" value="0.2" />
+  <xacro:property name="chassis_mass" value="5.0" />
+  <xacro:property name="drive_wheel_radius" value="0.1" />
+  <xacro:property name="drive_wheel_length" value="0.05" />
+  <xacro:property name="drive_wheel_mass" value="0.5" />
+  <xacro:property name="caster_wheel_radius" value="0.05" /> <xacro:property name="caster_wheel_mass" value="0.2" />
+  <xacro:property name="wheel_separation" value="${chassis_width / 2 + drive_wheel_length / 2}" />
+  <xacro:property name="drive_wheel_x_offset" value="-0.15" />
+  <xacro:property name="caster_wheel_x_offset" value="0.15" />
   <material name="chassis_color">
-    <color rgba="0.8 0.2 0.2 1"/> <!-- A lively red -->
+    <color rgba="0.8 0.2 0.2 1"/>
   </material>
   <material name="wheel_color">
-    <color rgba="0.1 0.1 0.1 1"/> <!-- Dark, like rubber -->
+    <color rgba="0.1 0.1 0.1 1"/>
   </material>
   <material name="camera_color">
-    <color rgba="0.0 0.0 1.0 1"/> <!-- Blue for the camera -->
-  </material>
-  <!-- Chassis / Base Link -->
+    <color rgba="0.0 0.0 1.0 1"/>
+  </material>
+  <material name="lidar_color">
+    <color rgba="0.1 0.8 0.8 1"/>
+  </material>
   <link name="base_link">
     <visual>
-      <origin xyz="0 0 0.3"/>
-      <geometry>
-        <box size="0.6 0.5 0.2"/>
+      <origin xyz="0 0 ${drive_wheel_radius}"/>
+      <geometry>
+        <box size="${chassis_length} ${chassis_width} ${chassis_height}"/>
       </geometry>
       <material name="chassis_color"/>
     </visual>
     <collision>
-      <origin xyz="0 0 0.3"/>
-      <geometry>
-        <box size="0.6 0.5 0.2"/>
-      </geometry>
-    </collision>
-    <inertial>
-      <origin xyz="0 0 0.3"/>
-      <mass value="5.0"/>
+      <origin xyz="0 0 ${drive_wheel_radius}"/>
+      <geometry>
+        <box size="${chassis_length} ${chassis_width} ${chassis_height}"/>
+      </geometry>
+    </collision>
+    <inertial>
+      <origin xyz="0 0 ${drive_wheel_radius}"/>
+      <mass value="${chassis_mass}"/>
       <inertia ixx="0.1" ixy="0" ixz="0" iyy="0.1" iyz="0" izz="0.1"/>
     </inertial>
@@ -35,127 +47,167 @@
     <material>Gazebo/Red</material>
   </gazebo>
-  <!-- Front Left Wheel -->
-  <link name="wheel_front_left">
-    <visual>
-      <geometry>
-        <cylinder radius="0.1" length="0.05"/>
-      </geometry>
-      <material name="wheel_color"/>
-    </visual>
-    <collision>
-      <geometry>
-        <cylinder radius="0.1" length="0.05"/>
-      </geometry>
-    </collision>
-    <inertial>
-      <mass value="0.5"/>
+  <link name="drive_wheel_left_link">
+    <visual>
+      <geometry>
+        <cylinder radius="${drive_wheel_radius}" length="${drive_wheel_length}"/>
+      </geometry>
+      <material name="wheel_color"/>
+    </visual>
+    <collision>
+      <geometry>
+        <cylinder radius="${drive_wheel_radius}" length="${drive_wheel_length}"/>
+      </geometry>
+    </collision>
+    <inertial>
+      <mass value="${drive_wheel_mass}"/>
       <inertia ixx="0.001" ixy="0" ixz="0" iyy="0.001" iyz="0" izz="0.001"/>
     </inertial>
   </link>
-  <gazebo reference="wheel_front_left">
-    <material>Gazebo/Black</material>
-  </gazebo>
-  <!-- Front Right Wheel -->
-  <link name="wheel_front_right">
-    <visual>
-      <geometry>
-        <cylinder radius="0.1" length="0.05"/>
-      </geometry>
-      <material name="wheel_color"/>
-    </visual>
-    <collision>
-      <geometry>
-        <cylinder radius="0.1" length="0.05"/>
-      </geometry>
-    </collision>
-    <inertial>
-      <mass value="0.5"/>
+  <gazebo reference="drive_wheel_left_link">
+    <material>Gazebo/Black</material>
+    <mu1>1.0</mu1>
+    <mu2>1.0</mu2>
+  </gazebo>
+  <link name="drive_wheel_right_link">
+    <visual>
+      <geometry>
+        <cylinder radius="${drive_wheel_radius}" length="${drive_wheel_length}"/>
+      </geometry>
+      <material name="wheel_color"/>
+    </visual>
+    <collision>
+      <geometry>
+        <cylinder radius="${drive_wheel_radius}" length="${drive_wheel_length}"/>
+      </geometry>
+    </collision>
+    <inertial>
+      <mass value="${drive_wheel_mass}"/>
       <inertia ixx="0.001" ixy="0" ixz="0" iyy="0.001" iyz="0" izz="0.001"/>
     </inertial>
   </link>
-  <gazebo reference="wheel_front_right">
-    <material>Gazebo/Black</material>
-  </gazebo>
-  <!-- Rear Left Wheel -->
-  <link name="wheel_rear_left">
-    <visual>
-      <geometry>
-        <cylinder radius="0.1" length="0.05"/>
-      </geometry>
-      <material name="wheel_color"/>
-    </visual>
-    <collision>
-      <geometry>
-        <cylinder radius="0.1" length="0.05"/>
-      </geometry>
-    </collision>
-    <inertial>
-      <mass value="0.5"/>
-      <inertia ixx="0.001" ixy="0" ixz="0" iyy="0.001" iyz="0" izz="0.001"/>
-    </inertial>
-  </link>
-  <gazebo reference="wheel_rear_left">
-    <material>Gazebo/Black</material>
-  </gazebo>
-  <!-- Rear Right Wheel -->
-  <link name="wheel_rear_right">
-    <visual>
-      <geometry>
-        <cylinder radius="0.1" length="0.05"/>
-      </geometry>
-      <material name="wheel_color"/>
-    </visual>
-    <collision>
-      <geometry>
-        <cylinder radius="0.1" length="0.05"/>
-      </geometry>
-    </collision>
-    <inertial>
-      <mass value="0.5"/>
-      <inertia ixx="0.001" ixy="0" ixz="0" iyy="0.001" iyz="0" izz="0.001"/>
-    </inertial>
-  </link>
-  <gazebo reference="wheel_rear_right">
-    <material>Gazebo/Black</material>
-  </gazebo>
-  <!-- Joints for the Four Wheels -->
-  <joint name="joint_wheel_front_left" type="continuous">
-    <origin xyz="0.3 0.25 0.1" rpy="-1.5708 0 0"/>
-    <parent link="base_link"/>
-    <child link="wheel_front_left"/>
-    <axis xyz="0 1 0"/>
-  </joint>
-  <joint name="joint_wheel_front_right" type="continuous">
-    <origin xyz="0.3 -0.25 0.1" rpy="-1.5708 0 0"/>
-    <parent link="base_link"/>
-    <child link="wheel_front_right"/>
-    <axis xyz="0 1 0"/>
-  </joint>
-  <joint name="joint_wheel_rear_left" type="continuous">
-    <origin xyz="-0.3 0.25 0.1" rpy="-1.5708 0 0"/>
-    <parent link="base_link"/>
-    <child link="wheel_rear_left"/>
-    <axis xyz="0 1 0"/>
-  </joint>
-  <joint name="joint_wheel_rear_right" type="continuous">
-    <origin xyz="-0.3 -0.25 0.1" rpy="-1.5708 0 0"/>
-    <parent link="base_link"/>
-    <child link="wheel_rear_right"/>
-    <axis xyz="0 1 0"/>
-  </joint>
-  <!-- Camera Link & Sensor Plugin -->
+  <gazebo reference="drive_wheel_right_link">
+    <material>Gazebo/Black</material>
+    <mu1>1.0</mu1>
+    <mu2>1.0</mu2>
+  </gazebo>
+  <link name="caster_wheel_left_link">
+    <visual>
+      <geometry>
+        <sphere radius="${caster_wheel_radius}"/>
+      </geometry>
+      <material name="wheel_color"/>
+    </visual>
+    <collision>
+      <geometry>
+        <sphere radius="${caster_wheel_radius}"/>
+      </geometry>
+    </collision>
+    <inertial>
+      <mass value="${caster_wheel_mass}"/>
+      <inertia ixx="0.0001" ixy="0" ixz="0" iyy="0.0001" iyz="0" izz="0.0001"/>
+    </inertial>
+  </link>
+  <gazebo reference="caster_wheel_left_link">
+    <material>Gazebo/Black</material>
+    <mu1>0.01</mu1>
+    <mu2>0.01</mu2>
+  </gazebo>
+  <link name="caster_wheel_right_link">
+    <visual>
+      <geometry>
+        <sphere radius="${caster_wheel_radius}"/>
+      </geometry>
+      <material name="wheel_color"/>
+    </visual>
+    <collision>
+      <geometry>
+        <sphere radius="${caster_wheel_radius}"/>
+      </geometry>
+    </collision>
+    <inertial>
+      <mass value="${caster_wheel_mass}"/>
+      <inertia ixx="0.0001" ixy="0" ixz="0" iyy="0.0001" iyz="0" izz="0.0001"/>
+    </inertial>
+  </link>
+  <gazebo reference="caster_wheel_right_link">
+    <material>Gazebo/Black</material>
+    <mu1>0.01</mu1>
+    <mu2>0.01</mu2>
+  </gazebo>
   <link name="camera_link">
     <visual>
-      <origin xyz="0 0 0"/>
-      <geometry>
-        <box size="0.1 0.1 0.1"/>
+      <geometry>
+        <box size="0.05 0.1 0.05"/>
       </geometry>
       <material name="camera_color"/>
     </visual>
   </link>
+  <link name="imu_link"/>
+  <link name="lidar_link">
+    <visual>
+      <geometry>
+        <cylinder radius="0.05" length="0.04"/>
+      </geometry>
+      <material name="lidar_color"/>
+    </visual>
+  </link>
+  <joint name="drive_wheel_left_joint" type="continuous">
+    <origin xyz="${drive_wheel_x_offset} ${wheel_separation} 0" rpy="-1.5708 0 0"/>
+    <parent link="base_link"/>
+    <child link="drive_wheel_left_link"/>
+    <axis xyz="0 0 1"/> </joint>
+  <joint name="drive_wheel_right_joint" type="continuous">
+    <origin xyz="${drive_wheel_x_offset} -${wheel_separation} 0" rpy="-1.5708 0 0"/>
+    <parent link="base_link"/>
+    <child link="drive_wheel_right_link"/>
+    <axis xyz="0 0 1"/>
+  </joint>
+  <joint name="caster_wheel_left_joint" type="fixed">
+    <origin xyz="${caster_wheel_x_offset} ${chassis_width/2 - 0.05} -${drive_wheel_radius - caster_wheel_radius}"/>
+    <parent link="base_link"/>
+    <child link="caster_wheel_left_link"/>
+  </joint>
+  <joint name="caster_wheel_right_joint" type="fixed">
+    <origin xyz="${caster_wheel_x_offset} -${chassis_width/2 - 0.05} -${drive_wheel_radius - caster_wheel_radius}"/>
+    <parent link="base_link"/>
+    <child link="caster_wheel_right_link"/>
+  </joint>
+  <joint name="camera_joint" type="fixed">
+    <origin xyz="${chassis_length/2} 0 ${drive_wheel_radius + chassis_height/2}" rpy="0 0 0"/>
+    <parent link="base_link"/>
+    <child link="camera_link"/>
+  </joint>
+  <joint name="imu_joint" type="fixed">
+    <origin xyz="0 0 ${drive_wheel_radius}"/>
+    <parent link="base_link"/>
+    <child link="imu_link"/>
+  </joint>
+  <joint name="lidar_joint" type="fixed">
+    <origin xyz="0 0 ${drive_wheel_radius + chassis_height + 0.02}"/>
+    <parent link="base_link"/>
+    <child link="lidar_link"/>
+  </joint>
+  <gazebo>
+    <plugin name="gazebo_ros_diff_drive" filename="libgazebo_ros_diff_drive.so">
+      <ros>
+        <namespace>/</namespace>
+        <remapping>cmd_vel:=/cmd_vel</remapping>
+      </ros>
+      <left_joint>drive_wheel_left_joint</left_joint>
+      <right_joint>drive_wheel_right_joint</right_joint>
+      <wheel_separation>${wheel_separation * 2}</wheel_separation>
+      <wheel_diameter>${drive_wheel_radius * 2}</wheel_diameter>
+      <max_wheel_torque>20</max_wheel_torque>
+      <max_wheel_acceleration>1.0</max_wheel_acceleration>
+      <update_rate>50</update_rate>
+      <odometry_topic>odom</odometry_topic>
+      <odometry_frame>odom</odometry_frame>
+      <robot_base_frame>base_link</robot_base_frame>
+      <publish_odometry_tf>true</publish_odometry_tf>
+      <publish_wheel_tf>false</publish_wheel_tf>
+    </plugin>
+  </gazebo>
   <gazebo reference="camera_link">
     <sensor type="camera" name="camera_sensor">
-      <pose>0 0 0 0 0 0</pose>
-      <always_on>true</always_on>
       <update_rate>30</update_rate>
       <camera>
@@ -170,32 +222,53 @@
           <far>100</far>
         </clip>
+        <noise>
+          <type>gaussian</type>
+          <mean>0.0</mean>
+          <stddev>0.007</stddev>
+        </noise>
       </camera>
       <plugin name="gazebo_ros_camera" filename="libgazebo_ros_camera.so">
-        <cameraName>camera</cameraName>
-        <frameName>camera_link</frameName>
+        <image_topic_name>/camera_sensor/image_raw</image_topic_name>
+        <camera_info_topic_name>/camera_sensor/camera_info</camera_info_topic_name>
+        <frame_name>camera_link</frame_name>
       </plugin>
     </sensor>
   </gazebo>
-  <!-- Updated Camera Joint: Now the camera is mounted forward without an unnecessary rotation -->
-  <joint name="camera_joint" type="fixed">
-    <origin xyz="0.2 0 0.5" rpy="0 0 0"/>
-    <parent link="base_link"/>
-    <child link="camera_link"/>
-  </joint>
-  <!-- Diff Drive Plugin Configuration -->
-  <gazebo reference="base_link">
-    <plugin name="gazebo_ros_diff_drive" filename="libgazebo_ros_diff_drive.so">
-      <ros>
-        <remapping>cmd_vel:=/cmd_vel</remapping>
-      </ros>
-      <left_joint>joint_wheel_front_left</left_joint>
-      <left_joint>joint_wheel_rear_left</left_joint>
-      <right_joint>joint_wheel_front_right</right_joint>
-      <right_joint>joint_wheel_rear_right</right_joint>
-      <wheel_separation>0.5</wheel_separation>
-      <wheel_diameter>0.2</wheel_diameter>
-      <update_rate>50</update_rate>
-      <torque>5.0</torque>
-    </plugin>
+  <gazebo reference="imu_link">
+    <sensor name="imu_sensor" type="imu">
+      <update_rate>100</update_rate>
+      <plugin filename="libgazebo_ros_imu_sensor.so" name="imu_plugin">
+        <ros>
+          <namespace>/imu</namespace>
+          <remapping>~/out:=data</remapping>
+        </ros>
+      </plugin>
+    </sensor>
+  </gazebo>
+  <gazebo reference="lidar_link">
+    <sensor type="ray" name="lidar_360">
+      <pose>0 0 0 0 0 0</pose>
+      <visualize>true</visualize>
+      <update_rate>10</update_rate>
+      <ray>
+        <scan>
+          <horizontal>
+            <samples>360</samples> <resolution>1</resolution>
+            <min_angle>-3.14159</min_angle>
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